File: Hardware/PCBLayout/LED-Board_PCBLayout.kicad_pcb (KiCad board)
At the start: 2 copper layers, 9 parts, among them U1 L78L05_TO92

Commit message: power supply
Parts:
- removed H1, H2: MountingHole_Pad, MountingHole:MountingHole_2.1mm
- D1, D2: footprint Diode_THT:D_DO-201_P12.70mm_Horizontal -> Diode_THT:D_DO-35_SOD27_P7.62mm_Horizontal
- moved D1 43.5 mm to (24.2, 24.0)
- moved D2 35.2 mm to (35.2, 24.0)
- moved C2 30.8 mm to (30.0, 28.0), turned to -90 degrees
- moved C1 26.1 mm to (25.0, 29.0)
- moved U1 22.4 mm to (35.0, 28.0), turned to 180 degrees
- moved C4 11.1 mm to (40.0, 29.0)
- moved C3 10.1 mm to (37.5, 28.0), turned to -90 degrees
Connections:
- U1 pad 2: GND -> unconnected-(U1-Pad2)
Routing:
- net GND: track 0.00 -> 2.75 mm

Commit message: power supply
Parts:
- added REF**: MountingHole_4.3mm_M4_DIN965, MountingHole:MountingHole_4.3mm_M4_DIN965, F.Cu at (24.0, 116.0)
- added REF**: MountingHole_4.3mm_M4_DIN965, MountingHole:MountingHole_4.3mm_M4_DIN965, F.Cu at (116.0, 24.0)
- added REF**: MountingHole_4.3mm_M4_DIN965, MountingHole:MountingHole_4.3mm_M4_DIN965, F.Cu at (24.0, 24.0)
- added REF**: MountingHole_4.3mm_M4_DIN965, MountingHole:MountingHole_4.3mm_M4_DIN965, F.Cu at (116.0, 116.0)
- moved C1 9.22 mm to (34.0, 31.0)
- moved C2 9.22 mm to (39.0, 30.0)
- moved C3 9.22 mm to (46.5, 30.0)
- moved C4 9.22 mm to (49.0, 31.0)
- moved D2 9.22 mm to (44.2, 26.0)
- moved U1 9.22 mm to (44.0, 30.0)
- moved D1 9.22 mm to (33.2, 26.0)
Connections:
- U1 pad 2: unconnected-(U1-Pad2) -> GND
Routing:
- net Net-(C1-Pad1): track 0.00 -> 27.3 mm
- net Net-(C3-Pad1): track 0.00 -> 10.1 mm
- net GND: track 2.75 -> 0.00 mm
Other:
- board outline added: 100 x 100 mm
- board text added: "LED-Board"
Changed lines of the file:
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@@
   )
   (paper "A4")
+  (title_block
+    (title "LED-Board")
+    (date "2022-06-27")
+    (rev "1.1")
+  )
   (layers
     (0 "F.Cu" signal)
@@
   (net 3 "Net-(C3-Pad1)")
   (net 4 "+12V")
-  (net 5 "unconnected-(U1-Pad2)")
   (footprint "Package_TO_SOT_THT:TO-92_Inline" (layer "F.Cu")
-    (at 35 28 180)
+    (at 44 30 180)
     (descr "TO-92 leads in-line, narrow, oval pads, drill 0.75mm (see NXP sot054_po.pdf)")
     (tags "to-92 sc-43 sc-43a sot54 PA33 transistor")
@@
       (net 3 "Net-(C3-Pad1)") (pinfunction "VO") (pintype "power_out"))
     (pad "2" thru_hole oval (at 1.27 0 180) (size 1.05 1.5) (drill 0.75) (layers *.Cu *.Mask)
-      (net 5 "unconnected-(U1-Pad2)") (pinfunction "GND") (pintype "power_in"))
+      (net 2 "GND") (pinfunction "GND") (pintype "power_in"))
     (pad "3" thru_hole oval (at 2.54 0 180) (size 1.05 1.5) (drill 0.75) (layers *.Cu *.Mask)
       (net 1 "Net-(C1-Pad1)") (pinfunction "VI") (pintype "power_in"))
@@
   )
   (footprint "Capacitor_THT:CP_Radial_D5.0mm_P2.50mm" (layer "F.Cu")
-    (at 25 29)
+    (at 34 31)
     (descr "CP, Radial series, Radial, pin pitch=2.50mm, , diameter=5mm, Electrolytic Capacitor")
     (tags "CP Radial series Radial pin pitch 2.50mm  diameter 5mm Electrolytic Capacitor")
@@
   )
   (footprint "Capacitor_THT:CP_Radial_D5.0mm_P2.50mm" (layer "F.Cu")
-    (at 40 29)
+    (at 49 31)
     (descr "CP, Radial series, Radial, pin pitch=2.50mm, , diameter=5mm, Electrolytic Capacitor")
     (tags "CP Radial series Radial pin pitch 2.50mm  diameter 5mm Electrolytic Capacitor")
@@
   )
   (footprint "Capacitor_SMD:C_0201_0603Metric_Pad0.64x0.40mm_HandSolder" (layer "F.Cu")
-    (at 37.5 28 -90)
+    (at 46.5 30 -90)
     (descr "Capacitor SMD 0201 (0603 Metric), square (rectangular) end terminal, IPC_7351 nominal with elongated pad for handsoldering. (Body size source: https://www.vishay.com/docs/20052/crcw0201e3.pdf), generated with kicad-footprint-generator")
     (tags "capacitor handsolder")
@@
     )
   )
+  (footprint "MountingHole:MountingHole_4.3mm_M4_DIN965" (layer "F.Cu")
+    (at 24 116)
+    (descr "Mounting Hole 4.3mm, no annular, M4, DIN965")
+    (tags "mounting hole 4.3mm no annular m4 din965")
+    (attr exclude_from_pos_files exclude_from_bom)
+    (fp_text reference "REF**" (at 0 0) (layer "F.SilkS")
+      (effects (font (size 1 1) (thickness 0.15)))
+    )
+    (fp_text value "MountingHole_4.3mm_M4_DIN965" (at 0 4.75) (layer "F.Fab")
+      (effects (font (size 1 1) (thickness 0.15)))
+    )
+    (fp_text user "${REFERENCE}" (at 0 0) (layer "F.Fab")
+      (effects (font (size 1 1) (thickness 0.15)))
+    )
+    (fp_circle (center 0 0) (end 3.75 0) (layer "Cmts.User") (width 0.15) (fill none))
+    (fp_circle (center 0 0) (end 4 0) (layer "F.CrtYd") (width 0.05) (fill none))
+    (pad "" np_thru_hole circle (at 0 0) (size 4.3 4.3) (drill 4.3) (layers *.Cu *.Mask))
+  )
+  (footprint "MountingHole:MountingHole_4.3mm_M4_DIN965" (layer "F.Cu")
+    (at 116 24)
+    (descr "Mounting Hole 4.3mm, no annular, M4, DIN965")
+    (tags "mounting hole 4.3mm no annular m4 din965")
+    (attr exclude_from_pos_files exclude_from_bom)
+    (fp_text reference "REF**" (at 0 0) (layer "F.SilkS")
+      (effects (font (size 1 1) (thickness 0.15)))
+    )
+    (fp_text value "MountingHole_4.3mm_M4_DIN965" (at 0 4.75) (layer "F.Fab")
+      (effects (font (size 1 1) (thickness 0.15)))
+    )
+    (fp_text user "${REFERENCE}" (at 0 0) (layer "F.Fab")
+      (effects (font (size 1 1) (thickness 0.15)))
+    )
+    (fp_circle (center 0 0) (end 3.75 0) (layer "Cmts.User") (width 0.15) (fill none))
+    (fp_circle (center 0 0) (end 4 0) (layer "F.CrtYd") (width 0.05) (fill none))
+    (pad "" np_thru_hole circle (at 0 0) (size 4.3 4.3) (drill 4.3) (layers *.Cu *.Mask))
+  )
   (footprint "Capacitor_SMD:C_0201_0603Metric_Pad0.64x0.40mm_HandSolder" (layer "F.Cu")
-    (at 30 28 -90)
+    (at 39 30 -90)
     (descr "Capacitor SMD 0201 (0603 Metric), square (rectangular) end terminal, IPC_7351 nominal with elongated pad for handsoldering. (Body size source: https://www.vishay.com/docs/20052/crcw0201e3.pdf), generated with kicad-footprint-generator")
     (tags "capacitor handsolder")
@@
   )
   (footprint "Diode_THT:D_DO-35_SOD27_P7.62mm_Horizontal" (layer "F.Cu")
-    (at 35.19 24)
+    (at 44.19 26)
     (descr "Diode, DO-35_SOD27 series, Axial, Horizontal, pin pitch=7.62mm, , length*diameter=4*2mm^2, , http://www.diodes.com/_files/packages/DO-35.pdf")
     (tags "Diode DO-35_SOD27 series Axial Horizontal pin pitch 7.62mm  length 4mm diameter 2mm")
@@
     )
   )
+  (footprint "MountingHole:MountingHole_4.3mm_M4_DIN965" (layer "F.Cu")
+    (at 24 24)
+    (descr "Mounting Hole 4.3mm, no annular, M4, DIN965")
+    (tags "mounting hole 4.3mm no annular m4 din965")
+    (attr exclude_from_pos_files exclude_from_bom)
+    (fp_text reference "REF**" (at 0 0) (layer "F.SilkS")
+      (effects (font (size 1 1) (thickness 0.15)))
+    )
+    (fp_text value "MountingHole_4.3mm_M4_DIN965" (at 0 4.75) (layer "F.Fab")
+      (effects (font (size 1 1) (thickness 0.15)))
+    )
+    (fp_text user "${REFERENCE}" (at 0 0) (layer "F.Fab")
+      (effects (font (size 1 1) (thickness 0.15)))
+    )
+    (fp_circle (center 0 0) (end 3.75 0) (layer "Cmts.User") (width 0.15) (fill none))
+    (fp_circle (center 0 0) (end 4 0) (layer "F.CrtYd") (width 0.05) (fill none))
+    (pad "" np_thru_hole circle (at 0 0) (size 4.3 4.3) (drill 4.3) (layers *.Cu *.Mask))
+  )
+  (footprint "MountingHole:MountingHole_4.3mm_M4_DIN965" (layer "F.Cu")
+    (at 116 116)
+    (descr "Mounting Hole 4.3mm, no annular, M4, DIN965")
+    (tags "mounting hole 4.3mm no annular m4 din965")
+    (attr exclude_from_pos_files exclude_from_bom)
+    (fp_text reference "REF**" (at 0 0) (layer "F.SilkS")
+      (effects (font (size 1 1) (thickness 0.15)))
+    )
+    (fp_text value "MountingHole_4.3mm_M4_DIN965" (at 0 4.75) (layer "F.Fab")
+      (effects (font (size 1 1) (thickness 0.15)))
+    )
+    (fp_text user "${REFERENCE}" (at 0 0) (layer "F.Fab")
+      (effects (font (size 1 1) (thickness 0.15)))
+    )
+    (fp_circle (center 0 0) (end 3.75 0) (layer "Cmts.User") (width 0.15) (fill none))
+    (fp_circle (center 0 0) (end 4 0) (layer "F.CrtYd") (width 0.05) (fill none))
+    (pad "" np_thru_hole circle (at 0 0) (size 4.3 4.3) (drill 4.3) (layers *.Cu *.Mask))
+  )
   (footprint "Diode_THT:D_DO-35_SOD27_P7.62mm_Horizontal" (layer "F.Cu")
-    (at 24.19 24)
+    (at 33.19 26)
     (descr "Diode, DO-35_SOD27 series, Axial, Horizontal, pin pitch=7.62mm, , length*diameter=4*2mm^2, , http://www.diodes.com/_files/packages/DO-35.pdf")
     (tags "Diode DO-35_SOD27 series Axial Horizontal pin pitch 7.62mm  length 4mm diameter 2mm")
@@
     )
   )
-  (gr_line (start 120 120) (end 20 120) (layer "F.Cu") (width 0.2))
-  (gr_line (start 20 20) (end 120 20) (layer "F.Cu") (width 0.2))
-  (gr_line (start 120 20) (end 120 120) (layer "F.Cu") (width 0.2))
-  (gr_line (start 20 120) (end 20 20) (layer "F.Cu") (width 0.2))
-  (segment (start 27.5 29) (end 29.4075 29) (width 0.5) (layer "F.Cu") (net 2))
-  (segment (start 29.4075 29) (end 30 28.4075) (width 0.5) (layer "F.Cu") (net 2))
+  (gr_line (start 120 20) (end 120 120) (layer "Edge.Cuts") (width 0.1))
+  (gr_line (start 20 120) (end 20 20) (layer "Edge.Cuts") (width 0.1))
+  (gr_line (start 120 120) (end 20 120) (layer "Edge.Cuts") (width 0.1))
+  (gr_line (start 20 20) (end 120 20) (layer "Edge.Cuts") (width 0.1))
+  (gr_text "LED-Board" (at 72 117) (layer "F.SilkS")
+    (effects (font (size 3 3) (thickness 0.3)))
+  )
+  (segment (start 42.81 24) (end 51 24) (width 0.5) (layer "F.Cu") (net 1))
+  (segment (start 38.4075 29) (end 39 29.5925) (width 0.5) (layer "F.Cu") (net 1))
+  (segment (start 51 24) (end 52 25) (width 0.5) (layer "F.Cu") (net 1))
+  (segment (start 52 25.81) (end 51.81 26) (width 0.5) (layer "F.Cu") (net 1))
+  (segment (start 40.81 26) (end 42.81 24) (width 0.5) (layer "F.Cu") (net 1))
+  (segment (start 41.0525 29.5925) (end 41.46 30) (width 0.5) (layer "F.Cu") (net 1))
+  (segment (start 34 31) (end 34 30) (width 0.5) (layer "F.Cu") (net 1))
+  (segment (start 52 25) (end 52 25.81) (width 0.5) (layer "F.Cu") (net 1))
+  (segment (start 40.81 26) (end 40.81 29.35) (width 0.5) (layer "F.Cu") (net 1))
+  (segment (start 35 29) (end 38.4075 29) (width 0.5) (layer "F.Cu") (net 1))
+  (segment (start 40.81 29.35) (end 41.46 30) (width 0.5) (layer "F.Cu") (net 1))
+  (segment (start 34 30) (end 35 29) (width 0.5) (layer "F.Cu") (net 1))
+  (segment (start 39 29.5925) (end 41.0525 29.5925) (width 0.5) (layer "F.Cu") (net 1))
+  (segment (start 52 25.81) (end 51.81 26) (width 0.5) (layer "B.Cu") (net 1))
+  (segment (start 44 30) (end 44.4075 29.5925) (width 0.5) (layer "F.Cu") (net 3))
+  (segment (start 47.5925 29.5925) (end 49 31) (width 0.5) (layer "F.Cu") (net 3))
+  (segment (start 46.5 29.5925) (end 47.5925 29.5925) (width 0.5) (layer "F.Cu") (net 3))
+  (segment (start 44 30) (end 44 26.19) (width 0.5) (layer "F.Cu") (net 3))
+  (segment (start 44 26.19) (end 44.19 26) (width 0.5) (layer "F.Cu") (net 3))
+  (segment (start 44.4075 29.5925) (end 46.5 29.5925) (width 0.5) (layer "F.Cu") (net 3))
+  (segment (start 44.19 29.81) (end 44 30) (width 0.5) (layer "B.Cu") (net 3))
   (zone (net 2) (net_name "GND") (layers F&B.Cu) (hatch edge 0.508)
     (connect_pads (clearance 0.508))
-    (min_thickness 0.254)
-    (fill (thermal_gap 0.508) (thermal_bridge_width 0.508))
+    (min_thickness 0.254) (filled_areas_thickness no)
+    (fill yes (thermal_gap 0.508) (thermal_bridge_width 0.508))
     (polygon
       (pts

Commit message: power supply / power unit
Parts:
- added  : Layer1, Pabst:Layer1, F.Cu at (32.0, 117.0)
- added  : Layer2, Pabst:Layer2, F.Cu at (32.0, 117.0)
- added D3: BZV55C3V3, Diode_SMD:D_MiniMELF, F.Cu at (41.0, 56.0)
- added GND1: MHole, Connector_Pin:Pin_D1.3mm_L11.0mm, F.Cu at (30.0, 59.0)
- added LED1: MHole, Connector_Pin:Pin_D1.3mm_L11.0mm, F.Cu at (30.0, 54.0)
- added Q1: BC846, Package_TO_SOT_SMD:SOT-23, F.Cu at (35.0, 59.0)
- added Q2: BC856, Package_TO_SOT_SMD:SOT-23, F.Cu at (35.0, 54.0)
- added R1: R_Small, Resistor_SMD:R_0201_0603Metric_Pad0.64x0.40mm_HandSolder, F.Cu at (41.4, 52.0)
- added R2: R_Small, Resistor_SMD:R_0201_0603Metric_Pad0.64x0.40mm_HandSolder, F.Cu at (42.4, 60.0)
- D1, D2: value DIODE -> 1N4006; footprint Diode_THT:D_DO-35_SOD27_P7.62mm_Horizontal -> Diode_THT:D_DO-41_SOD81_P10.16mm_Horizontal
- moved D1 11.1 mm to (44.1, 24.0), turned to 180 degrees
- moved C4 4.49 mm to (53.3, 29.7)
- moved D2 4.23 mm to (47.9, 24.0)
- moved C3 3.67 mm to (50.0, 28.9)
- moved U1 3.45 mm to (47.3, 29.0)
- moved C2 3.20 mm to (42.0, 28.9)
- moved C1 2.55 mm to (36.2, 29.7)
Connections:
- C1 pad 1: Net-(C1-Pad1) -> +12V
- C2 pad 1: Net-(C1-Pad1) -> +12V
- D1 pad 2: Net-(C1-Pad1) -> +12V
- D2 pad 1: Net-(C3-Pad1) -> +12V
- D2 pad 2: Net-(C1-Pad1) -> Net-(C3-Pad1)
- U1 pad 3: Net-(C1-Pad1) -> +12V
Routing:
- net Net-(C1-Pad1): track 27.3 -> 0.00 mm
- net Net-(C3-Pad1): track 10.1 -> 0.00 mm
Other:
- board text added: "LED-Board V1.1"
- board text removed: "LED-Board"
